File: testbench.brd (EAGLE design)
At the start: 100 x 100 mm, 45 parts, among them T1 C8492, T2 C8492, T3 C8545, T4 C8545, X1 MKDSN1,5/2-5,08

Commit message: text added and diodes defined
Parts:
- added R27, R28: 2k2, rcl:R0805
- D1, D2: value (none) -> C8062
Connections:
- net +3V3: now also R27.1, R28.1
- net D1: now also R28.2
- net D2: now also R27.2
Routing:
- net +3V3: track 116.1 -> 129.9 mm
- net D2: track 75.3 -> 85.2 mm
- net D1: track 71.9 -> 78.1 mm
