File: Testadapter/Testadapter.brd (EAGLE design)
At the start: 100 x 100 mm, 47 parts, among them T1 C8492, T2 C8492, T3 C8545, T4 C8545, X1 MKDSN1,5/2-5,08

Commit message: apply new folder structure, renamed files, stripped EAGLE lib for MEB connectors
Parts:
- JP1: device pinhead_own:2X11_MEB12S_MODULSEITE_SMD -> con-MEB:2X11_MEB12S_MODULSEITE_SMD
